File: pcb/KiBot-CICD-Template.kicad_sch (KiCad schematic)
At the start: 1 part

Commit message: update KiBot
Parts:
- removed LOGO1: Logo_Open_Hardware_Small, Symbol:OSHW-Symbol_6.7x6mm_SilkScreen, symbol Graphic:Logo_Open_Hardware_Small
Changed lines of the file:
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@@
   (title_block
     (title "KiBot-CICD-Template")
-    (date "%date%")
-    (rev "%version%")
+    (date "@date@")
+    (rev "@version@")
     (company "nerdyscout")
     (comment 4 "CERN Open Hardware Licence v2.0")
@@
   (symbol (lib_id "Graphic:Logo_Open_Hardware_Small") (at 274.32 175.26 0) (unit 1)
     (in_bom yes) (on_board yes)
-    (property "Reference" "LOGO1" (id 0) (at 274.32 168.275 0)
+    (property "Reference" "#LOGO1" (id 0) (at 274.32 168.275 0)
       (effects (font (size 1.27 1.27)) hide)
     )
@@
   (symbol_instances
     (path "/00000000-0000-0000-0000-00005e25fd05"
-      (reference "LOGO1") (unit 1) (value "Logo_Open_Hardware_Small") (footprint "Symbol:OSHW-Symbol_6.7x6mm_SilkScreen")
+      (reference "#LOGO1") (unit 1) (value "Logo_Open_Hardware_Small") (footprint "Symbol:OSHW-Symbol_6.7x6mm_SilkScreen")
     )
   )
